File: pcb/attinyx14/attinyx14_dev.kicad_pcb (KiCad board)
At the start: 2 copper layers, 22.6 x 62.2 mm, 28 parts, among them J1 USB_C_Receptacle_USB2.0_16P, J2 Conn_01x07, J3 Conn_01x07, J4 Conn_02x06, J5 Conn_01x02, J6 Conn_01x02, U1 USBLC6-2SC6, U2 ATtiny214-SS, U3 CH342K

Commit message: pcb layout done
Routing:
- net /PA4: track 0.00 -> 40.5 mm, vias 0 -> 2
- net /PB3: track 0.00 -> 37.2 mm
- net /PB2: track 0.00 -> 35.4 mm
- net /PA0: track 0.00 -> 32.6 mm
- net /PA3: track 0.00 -> 23.8 mm
- net /PB1: track 0.00 -> 23.2 mm
- net /PB0: track 0.00 -> 22.6 mm
- net /PA7: track 0.00 -> 21.4 mm
- net /PA1: track 0.00 -> 21.0 mm
- net /PA6: track 0.00 -> 20.1 mm
- net /PA2: track 0.00 -> 19.1 mm
- net /PA5: track 0.00 -> 18.9 mm
- net +5VA: track 17.8 -> 21.3 mm
Other:
- board size 22.6 x 62.2 mm -> 22.6 x 63.8 mm
